File: wxeda-sd-mod.sch (EAGLE design)
At the start: 26 parts, among them T1 2N3904, U1 SD_CARD, X1 TV OUT, X2 TAPE IN / OUT

Commit message: Added S-Video connector against RCA
Parts:
- removed R10: 150, SparkFun-Passives:RESISTORAXIAL-0.3
- removed R8: 1k, SparkFun-Passives:RESISTORAXIAL-0.3
- removed T1: 2N3904, transistor:2N3904
- removed X1: TV OUT, con-hirschmann:TOBU3
- added U$1: S-VIDEO, connectors-digital:MINIDIN_4
- C3: value 22n -> 47uF; device adafruit:C-US050-025X075 -> adafruit:CPOL-USE5-8.5
- R7: value 680 -> 75
- R9: value 51 -> 75
Connections:
- removed net N$2: R7.2, R8.1, T1.B
- removed net TVOUT: C3.2, C4.-, X1.1
- new net C_OUT: C4.-, U$1.4
- new net Y_OUT: C3.-, U$1.3
- net DSE: now also R7.1
- net DSEN4: now also R9.1; no longer R7.1
- net GND: now also U$1.1, U$1.2, U$1.CASE1, U$1.CASE2, U$1.SHIELDING; no longer R10.1, X1.2
- net N$7: now also C4.+, R9.2; no longer R9.1, T1.E
- net N$8: now also C3.+, R7.2; no longer C3.1, C4.+, R10.2, R9.2
- net VCC: no longer R8.2, T1.C
Other:
- moved on the sheet: C4, R7, R9
